Commit message: fixed pendulum rotation

File: flagpole.urdf (robot description, URDF)
Before this commit: robot flagpole, 6 links, 5 joints
Joints:
- joint pole_base_joint: axis 0.0 0.0 1.0 -> 0.0 1.0 0.0

Commit message: New Changes

File: flagpole.urdf (robot description, URDF)
Before this commit: robot flagpole, 6 links, 5 joints
Joints:
- joint pole_base_joint: limit (none) -> lower=-0.87266 upper=0.87266 effort=10.0 velocity=1.0; type continuous -> revolute
